Commit message: update README

File: piper_ros/piper_description/urdf/piper_description.urdf (robot description, URDF)
Before this commit: robot piper_description, 10 links, 9 joints
Links:
- link base_link: geometry collision mesh filename=/home/agilex/pika_ros/src/PikaAnyArm/piper_ros/piper_descri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; visual mesh filename=/home/agilex/pika_ros/src/PikaAnyArm/piper_ros/piper_descri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
- link gripper_base: geometry collision mesh filename=/home/agilex/pika_ros/src/PikaAnyArm/piper_ros/piper_descri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; visual mesh filename=/home/agilex/pika_ros/src/PikaAnyArm/piper_ros/piper_descri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
- link link1: geometry collision mesh filename=/home/agilex/pika_ros/src/PikaAnyArm/piper_ros/piper_descri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; visual mesh filename=/home/agilex/pika_ros/src/PikaAnyArm/piper_ros/piper_descri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
- link link2: geometry collision mesh filename=/home/agilex/pika_ros/src/PikaAnyArm/piper_ros/piper_descri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; visual mesh filename=/home/agilex/pika_ros/src/PikaAnyArm/piper_ros/piper_descri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
- link link3: geometry collision mesh filename=/home/agilex/pika_ros/src/PikaAnyArm/piper_ros/piper_descri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; visual mesh filename=/home/agilex/pika_ros/src/PikaAnyArm/piper_ros/piper_descri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
- link link4: geometry collision mesh filename=/home/agilex/pika_ros/src/PikaAnyArm/piper_ros/piper_descri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; visual mesh filename=/home/agilex/pika_ros/src/PikaAnyArm/piper_ros/piper_descri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
- link link5: geometry collision mesh filename=/home/agilex/pika_ros/src/PikaAnyArm/piper_ros/piper_descri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; visual mesh filename=/home/agilex/pika_ros/src/PikaAnyArm/piper_ros/piper_descri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
- link link6: geometry collision mesh filename=/home/agilex/pika_ros/src/PikaAnyArm/piper_ros/piper_descri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; visual mesh filename=/home/agilex/pika_ros/src/PikaAnyArm/piper_ros/piper_descri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
- link link7: geometry collision mesh filename=/home/agilex/pika_ros/src/PikaAnyArm/piper_ros/piper_descri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; visual mesh filename=/home/agilex/pika_ros/src/PikaAnyArm/piper_ros/piper_descri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
- link link8: geometry collision mesh filename=/home/agilex/pika_ros/src/PikaAnyArm/piper_ros/piper_descri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; visual mesh filename=/home/agilex/pika_ros/src/PikaAnyArm/piper_ros/piper_descri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

Commit message: update piper update joint1 limit

File: piper_ros/piper_description/urdf/piper_description.urdf (robot description, URDF)
Before this commit: robot piper_description, 10 links, 9 joints
Joints:
- joint joint1: limit lower=-2.618 upper=2.168 effort=100 velocity=5 -> lower=-2.618 upper=2.618 effort=100 velocity=5

Commit message: 修复了需要从绝对路径加载URDF的问题

File: piper_ros/piper_description/urdf/piper_description.urdf (robot description, URDF)
Before this commit: robot piper_description, 10 links, 9 joints
Links:
- link base_link: geometry collision mesh filename=package://piper_description/meshes/base_link.STL; visual mesh filename=package://piper_description/meshes/base_link.STL
- link gripper_base: geometry collision mesh filename=package://piper_description/meshes/gripper_base.STL; visual mesh filename=package://piper_description/meshes/gripper_base.STL
- link link1: geometry collision mesh filename=package://piper_description/meshes/link1.STL; visual mesh filename=package://piper_description/meshes/link1.STL
- link link2: geometry collision mesh filename=package://piper_description/meshes/link2.STL; visual mesh filename=package://piper_description/meshes/link2.STL
- link link3: geometry collision mesh filename=package://piper_description/meshes/link3.STL; visual mesh filename=package://piper_description/meshes/link3.STL
- link link4: geometry collision mesh filename=package://piper_description/meshes/link4.STL; visual mesh filename=package://piper_description/meshes/link4.STL
- link link5: geometry collision mesh filename=package://piper_description/meshes/link5.STL; visual mesh filename=package://piper_description/meshes/link5.STL
- link link6: geometry collision mesh filename=package://piper_description/meshes/link6.STL; visual mesh filename=package://piper_description/meshes/link6.STL
- link link7: geometry collision mesh filename=package://piper_description/meshes/link7.STL; visual mesh filename=package://piper_description/meshes/link7.STL
- link link8: geometry collision mesh filename=package://piper_description/meshes/link8.STL; visual mesh filename=package://piper_description/meshes/link8.STL
